Commit message: new_urdf_and_test

File: urdf/lm2/urdf/lm2.urdf (robot description, URDF)
Before this commit: robot lm2, 2 links, 1 joints
Links:
- link Link1: geometry collision mesh filename=../lm2/meshes/Link1.stl; visual mesh filename=../lm2/meshes/Link1.stl
- link base_link: geometry collision sphere radius=0.25; visual mesh filename=../meshes/base_link.stl
Joints:
- joint Joint1: limit lower=0 upper=0 effort=0 velocity=0 -> lower=0 upper=100 effort=100 velocity=100

File: urdf/zongzhuangURDF/urdf/zongzhuangURDF.urdf (robot description, URDF)
Before this commit: robot zongzhuangURDF, 13 links, 12 joints
Links:
- link L1: geometry collision mesh filename=../zongzhuangURDF/meshes/L1.stl; visual mesh filename=../zongzhuangURDF/meshes/L1.stl
- link L2: geometry collision mesh filename=../zongzhuangURDF/meshes/L2.stl; visual mesh filename=../zongzhuangURDF/meshes/L2.stl
- link L3: geometry collision mesh filename=../zongzhuangURDF/meshes/L3.stl; visual mesh filename=../zongzhuangURDF/meshes/L3.stl
- link L4: geometry collision mesh filename=../zongzhuangURDF/meshes/L4.stl; visual mesh filename=../zongzhuangURDF/meshes/L4.stl
- link L5: geometry collision mesh filename=../zongzhuangURDF/meshes/L5.stl; visual mesh filename=../zongzhuangURDF/meshes/L5.stl
- link L6: geometry collision mesh filename=../zongzhuangURDF/meshes/L6.stl; visual mesh filename=../zongzhuangURDF/meshes/L6.stl
- link R1: geometry collision mesh filename=../zongzhuangURDF/meshes/R1.stl; visual mesh filename=../zongzhuangURDF/meshes/R1.stl
- link R2: geometry collision mesh filename=../zongzhuangURDF/meshes/R2.stl; visual mesh filename=../zongzhuangURDF/meshes/R2.stl
- link R3: geometry collision mesh filename=../zongzhuangURDF/meshes/R3.stl; visual mesh filename=../zongzhuangURDF/meshes/R3.stl
- link R4: geometry collision mesh filename=../zongzhuangURDF/meshes/R4.stl; visual mesh filename=../zongzhuangURDF/meshes/R4.stl
- link R5: geometry collision mesh filename=../zongzhuangURDF/meshes/R5.stl; visual mesh filename=../zongzhuangURDF/meshes/R5.stl
- link R6: geometry collision mesh filename=../zongzhuangURDF/meshes/R6.stl; visual mesh filename=../zongzhuangURDF/meshes/R6.stl
- link base_link: geometry collision mesh filename=../zongzhuangURDF/meshes/base_link.stl; visual mesh filename=../zongzhuangURDF/meshes/base_link.stl
Joints:
- joint l1: limit lower=0 upper=0 effort=0 velocity=0 -> lower=0 upper=100 effort=100 velocity=100
- joint l2: limit lower=0 upper=0 effort=0 velocity=0 -> lower=0 upper=100 effort=100 velocity=100
- joint l3: limit lower=0 upper=0 effort=0 velocity=0 -> lower=0 upper=100 effort=100 velocity=100
- joint l4: limit lower=0 upper=0 effort=0 velocity=0 -> lower=0 upper=100 effort=100 velocity=100
- joint l5: limit lower=0 upper=0 effort=0 velocity=0 -> lower=0 upper=100 effort=100 velocity=100
- joint l6: limit lower=0 upper=0 effort=0 velocity=0 -> lower=0 upper=100 effort=100 velocity=100
- joint r1: limit lower=0 upper=0 effort=0 velocity=0 -> lower=0 upper=100 effort=100 velocity=100
- joint r2: limit lower=0 upper=0 effort=0 velocity=0 -> lower=0 upper=100 effort=100 velocity=100
- joint r3: limit lower=0 upper=0 effort=0 velocity=0 -> lower=0 upper=100 effort=100 velocity=100
- joint r4: limit lower=0 upper=0 effort=0 velocity=0 -> lower=0 upper=100 effort=100 velocity=100
- joint r5: limit lower=0 upper=0 effort=0 velocity=0 -> lower=0 upper=100 effort=100 velocity=100
- joint r6: limit lower=0 upper=0 effort=0 velocity=0 -> lower=0 upper=100 effort=100 velocity=100
