Commit message: new_urdf_test

File: urdf/zongzhuangURDF5/urdf/zongzhuangURDF5.urdf (robot description, URDF)
Before this commit: robot zongzhuangURDF5, 13 links, 12 joints
Joints:
- joint l1: limit lower=0 upper=0 effort=0 velocity=0 -> lower=0 upper=3.1415926 effort=1 velocity=1
- joint l2: limit lower=0 upper=0 effort=0 velocity=0 -> lower=0 upper=3.1415926 effort=1 velocity=1; origin xyz=0 0 0 rpy=3.1416 -1.5708 0 -> xyz=0 0 0 rpy=0 -1.5708 0
- joint l3: limit lower=0 upper=0 effort=0 velocity=0 -> lower=0 upper=3.1415926 effort=1 velocity=1
- joint l4: limit lower=0 upper=0 effort=0 velocity=0 -> lower=0 upper=3.1415926 effort=1 velocity=1
- joint l5: limit lower=0 upper=0 effort=0 velocity=0 -> lower=0 upper=3.1415926 effort=1 velocity=1
- joint l6: limit lower=0 upper=0 effort=0 velocity=0 -> lower=0 upper=3.1415926 effort=1 velocity=1
- joint r1: limit lower=0 upper=0 effort=0 velocity=0 -> lower=0 upper=3.1415926 effort=1 velocity=1
- joint r2: limit lower=0 upper=0 effort=0 velocity=0 -> lower=0 upper=3.1415926 effort=1 velocity=1; origin xyz=0 0 0 rpy=3.1416 -1.5708 0 -> xyz=0 0 0 rpy=0 -1.5708 0
- joint r3: limit lower=0 upper=0 effort=0 velocity=0 -> lower=0 upper=3.1415926 effort=1 velocity=1
- joint r4: limit lower=0 upper=0 effort=0 velocity=0 -> lower=0 upper=3.1415926 effort=1 velocity=1
- joint r5: limit lower=0 upper=0 effort=0 velocity=0 -> lower=0 upper=3.1415926 effort=1 velocity=1
- joint r6: limit lower=0 upper=0 effort=0 velocity=0 -> lower=0 upper=3.1415926 effort=1 velocity=1

Commit message: 2023/12/8

File: urdf/zongzhuangURDF5/urdf/zongzhuangURDF5.urdf (robot description, URDF)
Before this commit: robot zongzhuangURDF5, 13 links, 12 joints
Joints:
- joint l1: limit lower=0 upper=3.1415926 effort=1 velocity=1 -> lower=0 upper=3.1415926 effort=500 velocity=1
- joint l2: limit lower=0 upper=3.1415926 effort=1 velocity=1 -> lower=0 upper=3.1415926 effort=500 velocity=1
- joint l3: limit lower=0 upper=3.1415926 effort=1 velocity=1 -> lower=0 upper=3.1415926 effort=500 velocity=1
- joint l4: limit lower=0 upper=3.1415926 effort=1 velocity=1 -> lower=0 upper=3.1415926 effort=500 velocity=1
- joint l5: limit lower=0 upper=3.1415926 effort=1 velocity=1 -> lower=0 upper=3.1415926 effort=500 velocity=1
- joint l6: limit lower=0 upper=3.1415926 effort=1 velocity=1 -> lower=0 upper=3.1415926 effort=500 velocity=1
- joint r1: limit lower=0 upper=3.1415926 effort=1 velocity=1 -> lower=0 upper=3.1415926 effort=500 velocity=1
- joint r2: limit lower=0 upper=3.1415926 effort=1 velocity=1 -> lower=0 upper=3.1415926 effort=500 velocity=1
- joint r3: limit lower=0 upper=3.1415926 effort=1 velocity=1 -> lower=0 upper=3.1415926 effort=500 velocity=1
- joint r4: limit lower=0 upper=3.1415926 effort=1 velocity=1 -> lower=0 upper=3.1415926 effort=500 velocity=1
- joint r5: limit lower=0 upper=3.1415926 effort=1 velocity=1 -> lower=0 upper=3.1415926 effort=500 velocity=1
- joint r6: limit lower=0 upper=3.1415926 effort=1 velocity=1 -> lower=0 upper=3.1415926 effort=500 velocity=1

Commit message: urdf更改

File: urdf/zongzhuangURDF5/urdf/zongzhuangURDF5.urdf (robot description, URDF)
Before this commit: robot zongzhuangURDF5, 13 links, 12 joints
Links:
- link L1: mass 1.54071073617692 -> 1.51779481990376
- link L2: mass 3.97430335027074 -> 3.59389626425694
- link L3: mass 3.65189106558222 -> 3.65910111444716
- link L4: mass 3.03366312440795 -> 2.85321169527239
- link L5: mass 0.118789875656532 -> 0.113692025844553
- link L6: mass 2.4373117048765 -> 2.40125862032741
