Commit message: 2024.2.27

File: urdf/SIAT/SIAT.urdf (robot description, URDF)
Before this commit: robot SIAT, 13 links, 12 joints
Joints:
- joint joint_l_5: limit lower=-0.62831 upper=0.69813 effort=200 velocity=10 -> lower=-0.62831 upper=0.69813 effort=300 velocity=10
- joint joint_l_6: limit lower=-0.34907 upper=0.43633 effort=200 velocity=10 -> lower=-0.34907 upper=0.43633 effort=300 velocity=10
- joint joint_r_4: limit lower=-0.052399 upper=1.2217 effort=200 velocity=10 -> lower=-0.052399 upper=1.2217 effort=300 velocity=10
- joint joint_r_5: limit lower=-0.62831 upper=0.69813 effort=200 velocity=10 -> lower=-0.62831 upper=0.69813 effort=300 velocity=10
- joint joint_r_6: limit lower=-0.43633 upper=0.34907 effort=200 velocity=10 -> lower=-0.43633 upper=0.34907 effort=300 velocity=10

Commit message: 2024.2.28

File: urdf/SIAT/SIAT.urdf (robot description, URDF)
Before this commit: robot SIAT, 13 links, 12 joints
Links:
- link l_1: geometry visual mesh filename=package://SIAT/meshes/l_1.STL
- link l_2: geometry visual mesh filename=package://SIAT/meshes/l_2.STL
- link l_3: geometry visual mesh filename=package://SIAT/meshes/l_3.STL
- link l_4: geometry visual mesh filename=package://SIAT/meshes/l_4.STL
- link l_5: geometry visual mesh filename=package://SIAT/meshes/l_5.STL
- link r_1: geometry visual mesh filename=package://SIAT/meshes/r_1.STL
- link r_2: geometry visual mesh filename=package://SIAT/meshes/r_2.STL
- link r_3: geometry visual mesh filename=package://SIAT/meshes/r_3.STL
- link r_4: geometry visual mesh filename=package://SIAT/meshes/r_4.STL
- link r_5: geometry visual mesh filename=package://SIAT/meshes/r_5.STL

Commit message: gait

File: urdf/SIAT/SIAT.urdf (robot description, URDF)
Before this commit: robot SIAT, 13 links, 12 joints
Joints:
- joint joint_l_1: axis 0 0 -1 -> 0 0 1
- joint joint_l_2: axis 0 0 -1 -> 0 0 1
- joint joint_l_3: axis 0 0 -1 -> 0 0 1
- joint joint_l_4: axis 0 0 -1 -> 0 0 1
- joint joint_l_5: axis 0 0 -1 -> 0 0 1; limit lower=-0.62831 upper=0.69813 effort=300 velocity=10 -> lower=-0.62831 upper=0.69813 effort=3000 velocity=10
- joint joint_r_1: axis 0 0 -1 -> 0 0 1
- joint joint_r_2: axis 0 0 -1 -> 0 0 1
- joint joint_r_5: limit lower=-0.62831 upper=0.69813 effort=300 velocity=10 -> lower=-0.62831 upper=0.69813 effort=3000 velocity=10
- joint joint_r_6: axis 0 0 -1 -> 0 0 1

Commit message: 2024.3.2

File: urdf/SIAT/SIAT.urdf (robot description, URDF)
Before this commit: robot SIAT, 13 links, 12 joints
Joints:
- joint joint_l_1: limit lower=-0.69813 upper=0.5236 effort=300 velocity=10 -> lower=-0.69813 upper=0.5236 effort=500 velocity=40
- joint joint_l_2: limit lower=-0.5236 upper=0.38397 effort=300 velocity=10 -> lower=-0.5236 upper=0.38397 effort=500 velocity=40
- joint joint_l_3: limit lower=-0.69813 upper=0.2618 effort=300 velocity=10 -> lower=-0.69813 upper=0.2618 effort=500 velocity=40
- joint joint_l_4: limit lower=-0.052399 upper=1.2217 effort=300 velocity=10 -> lower=-0.052399 upper=1.2217 effort=500 velocity=40
- joint joint_l_5: limit lower=-0.62831 upper=0.69813 effort=3000 velocity=10 -> lower=-0.62831 upper=0.69813 effort=3000 velocity=40
- joint joint_l_6: limit lower=-0.34907 upper=0.43633 effort=300 velocity=10 -> lower=-0.34907 upper=0.43633 effort=500 velocity=40
- joint joint_r_1: limit lower=-0.5236 upper=0.69813 effort=300 velocity=10 -> lower=-0.5236 upper=0.69813 effort=500 velocity=40
- joint joint_r_2: limit lower=-0.38397 upper=0.5236 effort=300 velocity=10 -> lower=-0.38397 upper=0.5236 effort=500 velocity=40
- joint joint_r_3: limit lower=-0.69813 upper=0.2618 effort=300 velocity=10 -> lower=-0.69813 upper=0.2618 effort=500 velocity=40
- joint joint_r_4: limit lower=-0.052399 upper=1.2217 effort=300 velocity=10 -> lower=-0.052399 upper=1.2217 effort=500 velocity=40
- joint joint_r_5: limit lower=-0.62831 upper=0.69813 effort=3000 velocity=10 -> lower=-0.62831 upper=0.69813 effort=3000 velocity=40
- joint joint_r_6: limit lower=-0.43633 upper=0.34907 effort=300 velocity=10 -> lower=-0.43633 upper=0.34907 effort=500 velocity=40

Commit message: 3.12

File: urdf/SIAT/SIAT.urdf (robot description, URDF)
Before this commit: robot SIAT, 13 links, 12 joints
Links:
- removed link r_1
- removed link r_2
- removed link r_3
- removed link r_4
- removed link r_5
- removed link r_6
- added link ar_1, mass 2.8322; visual mesh filename=package://SIAT/meshes/r_1.STL
- added link ar_2, mass 4.2266; visual mesh filename=package://SIAT/meshes/r_2.STL
- added link ar_3, mass 11.84; visual mesh filename=package://SIAT/meshes/r_3.STL
- added link ar_4, mass 3.321; visual mesh filename=package://SIAT/meshes/r_4.STL
- added link ar_5, mass 0.11725; visual mesh filename=package://SIAT/meshes/r_5.STL
- added link ar_6, mass 1.4525; collision mesh filename=package://SIAT/meshes/r_6.STL; visual mesh filename=package://SIAT/meshes/r_6.STL
Joints:
- removed joint joint_r_1
- removed joint joint_r_2
- removed joint joint_r_3
- removed joint joint_r_4
- removed joint joint_r_5
- removed joint joint_r_6
- added joint joint_ar_1: type revolute, parent base_link, child ar_1, origin xyz=0 0.105 0 rpy=1.5708 0 1.5708, axis 0 0 1, limit lower=-0.5236 upper=0.69813 effort=500 velocity=40
- added joint joint_ar_2: type revolute, parent ar_1, child ar_2, origin xyz=0.159 0 0 rpy=-1.5708 -1.5708 0, axis 0 0 1, limit lower=-0.38397 upper=0.5236 effort=500 velocity=40
- added joint joint_ar_3: type revolute, parent ar_2, child ar_3, origin xyz=0.205 0 0 rpy=-1.5708 1.5708 0, axis 0 0 1, limit lower=-0.69813 upper=0.2618 effort=500 velocity=40
- added joint joint_ar_4: type revolute, parent ar_3, child ar_4, origin xyz=0.44 0 0 rpy=0 0 0, axis 0 0 1, limit lower=-0.052399 upper=1.2217 effort=500 velocity=40
- added joint joint_ar_5: type revolute, parent ar_4, child ar_5, origin xyz=0.4 0 0 rpy=0 0 0, axis 0 0 1, limit lower=-0.62831 upper=0.69813 effort=3000 velocity=40
- added joint joint_ar_6: type revolute, parent ar_5, child ar_6, origin xyz=0 0 -0.0275 rpy=1.5708 0 0, axis 0 0 1, limit lower=-0.43633 upper=0.34907 effort=500 velocity=40
