Commit message: 0402

File: urdf/SIAT01/urdf/SIAT01.urdf (robot description, URDF)
Before this commit: robot SIAT01, 13 links, 12 joints
Links:
- link ar_1: geometry collision mesh filename=/home/leovento/Robot-learning/urdf/SIAT01/meshes/r_1.STL; visual mesh filename=/home/leovento/Robot-learning/urdf/SIAT01/meshes/r_1.STL
- link ar_2: geometry collision mesh filename=/home/leovento/Robot-learning/urdf/SIAT01/meshes/r_2.STL; visual mesh filename=/home/leovento/Robot-learning/urdf/SIAT01/meshes/r_2.STL
- link ar_3: geometry collision mesh filename=/home/leovento/Robot-learning/urdf/SIAT01/meshes/r_3.STL; visual mesh filename=/home/leovento/Robot-learning/urdf/SIAT01/meshes/r_3.STL
- link ar_4: geometry collision mesh filename=/home/leovento/Robot-learning/urdf/SIAT01/meshes/r_4.STL; visual mesh filename=/home/leovento/Robot-learning/urdf/SIAT01/meshes/r_4.STL
- link ar_5: geometry collision mesh filename=/home/leovento/Robot-learning/urdf/SIAT01/meshes/r_5.STL; visual mesh filename=/home/leovento/Robot-learning/urdf/SIAT01/meshes/r_5.STL
- link ar_6: geometry collision mesh filename=/home/leovento/Robot-learning/urdf/SIAT01/meshes/r_6.STL; visual mesh filename=/home/leovento/Robot-learning/urdf/SIAT01/meshes/r_6.STL
- link base_link: geometry collision mesh filename=/home/leovento/Robot-learning/urdf/SIAT01/meshes/base_link.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; visual mesh filename=/home/leovento/Robot-learning/urdf/SIAT01/meshes/base_link.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
- link l_1: geometry collision mesh filename=/home/leovento/Robot-learning/urdf/SIAT01/meshes/l_1.STL; visual mesh filename=/home/leovento/Robot-learning/urdf/SIAT01/meshes/l_1.STL
- link l_2: geometry collision mesh filename=/home/leovento/Robot-learning/urdf/SIAT01/meshes/l_2.STL; visual mesh filename=/home/leovento/Robot-learning/urdf/SIAT01/meshes/l_2.STL
- link l_3: geometry collision mesh filename=/home/leovento/Robot-learning/urdf/SIAT01/meshes/l_3.STL; visual mesh filename=/home/leovento/Robot-learning/urdf/SIAT01/meshes/l_3.STL
- link l_4: geometry collision mesh filename=/home/leovento/Robot-learning/urdf/SIAT01/meshes/l_4.STL; visual mesh filename=/home/leovento/Robot-learning/urdf/SIAT01/meshes/l_4.STL
- link l_5: geometry collision mesh filename=/home/leovento/Robot-learning/urdf/SIAT01/meshes/l_5.STL; visual mesh filename=/home/leovento/Robot-learning/urdf/SIAT01/meshes/l_5.STL
- link l_6: geometry collision mesh filename=/home/leovento/Robot-learning/urdf/SIAT01/meshes/l_6.STL; visual mesh filename=/home/leovento/Robot-learning/urdf/SIAT01/meshes/l_6.STL
